File: KeyBoard.kicad_sch (KiCad schematic)
At the start: 486 parts, among them J1 USB_C_Receptacle_USB2.0, J2 Epaper Display, J3 JTAG, J4 Battery, Q1 ZVN3306F, Q2 2N7002, Q3 AO3400A, Q4 2N7002, SW1 RESET, SW10 MX_SW_solder, SW100 MX_SW_solder, SW101 MX_SW_solder, SW102 MX_SW_solder, SW103 MX_SW_solder, SW104 MX_SW_solder, SW105 PWR, SW11 MX_SW_solder, SW12 MX_SW_solder, SW13 MX_SW_solder, SW14 MX_SW_solder, SW15 MX_SW_solder, SW16 MX_SW_solder, SW17 MX_SW_solder, SW18 MX_SW_solder, SW19 MX_SW_solder, SW2 MX_SW_solder, SW20 MX_SW_solder, SW21 MX_SW_solder, SW22 MX_SW_solder, SW23 MX_SW_solder, SW24 MX_SW_solder, SW25 MX_SW_solder, SW26 MX_SW_solder, SW27 MX_SW_solder, SW28 MX_SW_solder, SW29 MX_SW_solder, SW3 MX_SW_solder, SW30 MX_SW_solder, SW31 MX_SW_solder, SW32 MX_SW_solder, SW33 MX_SW_solder, SW34 MX_SW_solder, SW35 MX_SW_solder, SW36 MX_SW_solder, SW37 MX_SW_solder, SW38 MX_SW_solder, SW39 MX_SW_solder, SW4 MX_SW_solder, SW40 MX_SW_solder, SW41 MX_SW_solder, SW42 MX_SW_solder, SW43 MX_SW_solder, SW44 MX_SW_solder, SW45 MX_SW_solder, SW46 MX_SW_solder, SW47 MX_SW_solder, SW48 MX_SW_solder, SW49 MX_SW_solder, SW5 MX_SW_solder, SW50 MX_SW_solder, SW51 MX_SW_solder, SW52 MX_SW_solder, SW53 MX_SW_solder, SW54 MX_SW_solder, SW55 MX_SW_solder, SW56 MX_SW_solder, SW57 MX_SW_solder, SW58 MX_SW_solder, SW59 MX_SW_solder, SW6 MX_SW_solder, SW60 MX_SW_solder, SW61 MX_SW_solder, SW62 MX_SW_solder, SW63 MX_SW_solder, SW64 MX_SW_solder, SW65 MX_SW_solder, SW66 MX_SW_solder, SW67 MX_SW_solder, SW68 MX_SW_solder, SW69 MX_SW_solder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

Commit message: updated prokect
Parts:
- removed J2: Epaper Display, Connector_FFC-FPC:Hirose_FH12-24S-0.5SH_1x24-1MP_P0.50mm_Horizontal, symbol Connector:Conn_01x24_Female
- added J2: Conn_01x24_Socket, symbol Connector:Conn_01x24_Socket
- D110, D111, D112, D113, D114, D116, D117, D118, D119, D120, D122, D123, D124, D125, D126, D128, D129, D130, D131, D132, D134, D135, D136, D137, D138, D140, D141, D142, D143, D144, D146, D147, D148, D149, D150, D152, D153, D154, D155, D156, D158, D159, D160, D161, D162, D164, D165, D166, D167, D168, D170, D171, D172, D173, D174, D176, D177, D178, D179, D180, D182, D183, D184, D185, D186, D188, D189, D190, D191, D192, D194, D195, D196, D197, D198, D200, D201, D202, D203, D204, D206, D207, D208, D209, D210, D212, D213, D214, D215, D216, D218, D219, D220, D221, D224, D225, D226, D227, D229, D230, D231, D232: footprint marbastlib-mx:LED_MX_6028R_backMount -> LED_SMD:LED_WS2812B-MINI_PLCC4_3.5x3.5mm_P1.75mm
- U7: footprint Package_TO_SOT_SMD:SOT-23 -> Package_TO_SOT_SMD:SOT-23-3
Connections:
- net +3V3: now also J2.16 (Pin_16)
- net EPD_BUSY: now also J2.9 (Pin_9)
- net EPD_CS: now also J2.12 (Pin_12)
- net EPD_DC: now also J2.11 (Pin_11)
- net EPD_DIN: now also J2.14 (Pin_14)
- net EPD_RST: now also J2.10 (Pin_10)
- net EPD_SCK: now also J2.13 (Pin_13)
- net GDR: now also J2.2 (Pin_2)
- net GND: now also J2.17 (Pin_17)
- net PREVGH: now also J2.21 (Pin_21)
- net PREVGL: now also J2.23 (Pin_23)
- net RESE: now also J2.3 (Pin_3)
- net at C3.1: now also J2.5 (Pin_5)
- net at C2.1: now also J2.4 (Pin_4)
- net at C7.1: now also J2.20 (Pin_20)
- net at C4.1: now also J2.15 (Pin_15)
- net at C5.1: now also J2.18 (Pin_18)
- net at C6.1: now also J2.19 (Pin_19)
- net at C9.1: now also J2.22 (Pin_22)
- net at C11.1: now also J2.24 (Pin_24)
- net at JP1.1 (A), JP2.1 (A): now also J2.8 (Pin_8)

Commit message: updated project
Parts:
- removed C10, C11, C14, C18, C2, C3, C4, C5, C6, C7, C8, C9: 4.7uF, Capacitor_SMD:C_1210_3225Metric, symbol pspice:CAP
- removed J3: JTAG, Connector_PinHeader_2.54mm:PinHeader_1x05_P2.54mm_Vertical, symbol Connector:Conn_01x05_Female
- added C100, C101, C116, C121, C92, C93, C94, C95, C96, C97, C98, C99: 4.7uF, Capacitor_SMD:C_1210_3225Metric, symbol Device:C_Small
- added J2: Conn_01x05_Pin, Connector_PinHeader_2.54mm:PinHeader_1x05_P2.54mm_Vertical, symbol Connector:Conn_01x05_Pin
- J4: renamed from J2; footprint (none) -> Connector_FFC-FPC:Hirose_FH12-24S-0.5SH_1x24-1MP_P0.50mm_Horizontal
- renumbered C34 to C10, C121 to C102, C122 to C103, C123 to C104, C124 to C105, C125 to C106, C127 to C107, C128 to C108, C129 to C109, C35 to C11, C130 to C110, C131 to C111, C133 to C112, C134 to C113, C135 to C114, C136 to C115, C139 to C117, C140 to C118, C141 to C119, C37 to C12, C142 to C120, C144 to C122, C145 to C123, C146 to C124, C147 to C125, C38 to C13, C39 to C14, C40 to C15, C41 to C16, C43 to C17, C44 to C18, C45 to C19, C25 to C2, C46 to C20, C47 to C21, C15 to C22, C49 to C23, C50 to C24, C51 to C25, C52 to C26, C53 to C27, C55 to C28, C56 to C29, C26 to C3, C57 to C30, C58 to C31, C59 to C32, C17 to C33, C61 to C34, C62 to C35, C63 to C36, C64 to C37, C65 to C38, C67 to C39, C27 to C4, C68 to C40, C69 to C41, C70 to C42, C71 to C43, C73 to C44, C74 to C45, C75 to C46, C76 to C47, C77 to C48, C20 to C49, C28 to C5, C21 to C50, C79 to C51, C80 to C52, C81 to C53, C82 to C54, C83 to C55, C22 to C56, C85 to C57, C86 to C58, C87 to C59, C29 to C6, C88 to C60, C89 to C61, C23 to C62, C24 to C63, C91 to C64, C92 to C65, C93 to C66, C94 to C67, C95 to C68, C12 to C69, C31 to C7, C97 to C70, C98 to C71, C99 to C72, C100 to C73, C101 to C74, C103 to C75, C104 to C76, C105 to C77, C106 to C78, C107 to C79, C32 to C8, C109 to C80, C110 to C81, C111 to C82, C112 to C83, C113 to C84, C13 to C85, C16 to C86, C115 to C87, C116 to C88, C117 to C89, C33 to C9, C118 to C90, C119 to C91, D119 to D10, D162 to D100, D61 to D101, D62 to D102, D63 to D103, D64 to D104, D65 to D105, D66 to D106, D67 to D107, D68 to D108, D69 to D109, D120 to D11, D70 to D110, D71 to D111, D72 to D112, D164 to D113, D165 to D114, D166 to D115, D167 to D116, D168 to D117, D73 to D118, D74 to D119, D122 to D12, D75 to D120, D76 to D121, D77 to D122, D78 to D123, D79 to D124, D80 to D125, D81 to D126, D82 to D127, D83 to D128, D84 to D129, D123 to D13, D85 to D130, D86 to D131, D87 to D132, D88 to D133, D89 to D134, D170 to D135, D171 to D136, D172 to D137, D173 to D138, D174 to D139, D124 to D14, D90 to D140, D91 to D141, D92 to D142, D176 to D143, D177 to D144, D178 to D145, D179 to D146, D180 to D147, D182 to D148, D183 to D149, D125 to D15, D184 to D150, D185 to D151, D186 to D152, D93 to D153, D94 to D154, D95 to D155, D96 to D156, D97 to D157, D188 to D158, D189 to D159, D126 to D16, D190 to D160, D191 to D161, D192 to D162, D98 to D163, D99 to D164, D100 to D165, D101 to D166, D102 to D167, D103 to D168, D104 to D169, D128 to D17, D105 to D170, D106 to D171, D194 to D172, D195 to D173, D196 to D174, D197 to D175, D198 to D176, D107 to D177, D108 to D178, D109 to D179, D129 to D18, D200 to D180, D201 to D181, D202 to D182, D203 to D183, D204 to D184, D206 to D185, D207 to D186, D208 to D187, D209 to D188, D210 to D189, D130 to D19, D212 to D190, D213 to D191, D214 to D192, D215 to D193, D216 to D194, D218 to D195, D219 to D196, D220 to D197, D221 to D198, D224 to D199, D110 to D2, D131 to D20, D225 to D200, D226 to D201, D227 to D202, D28 to D203, D35 to D204, D48 to D205, D229 to D206, D230 to D207, D231 to D208, D232 to D209, D132 to D21, D134 to D22, D135 to D23, D136 to D24, D137 to D25, D138 to D26, D4 to D27, D5 to D28, D6 to D29, D111 to D3, D7 to D30, D8 to D31, D9 to D32, D10 to D33, D11 to D34, D12 to D35, D13 to D36, D14 to D37, D15 to D38, D140 to D39, D112 to D4, D141 to D40, D142 to D41, D143 to D42, D144 to D43, D16 to D44, D17 to D45, D18 to D46, D19 to D47, D20 to D48, D21 to D49, D113 to D5, D22 to D50, D23 to D51, D24 to D52, D25 to D53, D26 to D54, D27 to D55, D146 to D56, D147 to D57, D148 to D58, D149 to D59, D114 to D6, D150 to D60, D29 to D61, D30 to D62, D31 to D63, D32 to D64, D33 to D65, D34 to D66, D36 to D67, D37 to D68, D38 to D69, D116 to D7, D39 to D70, D40 to D71, D41 to D72, D152 to D73, D153 to D74, D154 to D75, D155 to D76, D156 to D77, D42 to D78, D43 to D79, D117 to D8, D44 to D80, D45 to D81, D46 to D82, D47 to D83, D49 to D84, D50 to D85, D51 to D86, D52 to D87, D53 to D88, D54 to D89, D118 to D9, D55 to D90, D56 to D91, D57 to D92, D58 to D93, D59 to D94, D60 to D95, D158 to D96, D159 to D97, D160 to D98, D161 to D99, J4 to J3, JP3 to JP1, JP1 to JP2, JP2 to JP3, Q2 to Q1, Q3 to Q2, Q4 to Q3, Q1 to Q4, R11 to R10, R12 to R11, R14 to R12, R15 to R13, R16 to R14, R17 to R15, R18 to R16, R19 to R17, R8 to R18, R13 to R19, R6 to R4, R7 to R5, R10 to R6, R4 to R7, R5 to R8, SW2 to SW1, SW11 to SW10, SW12 to SW11, SW13 to SW12, SW14 to SW13, SW15 to SW14, SW16 to SW15, SW17 to SW16, SW18 to SW17, SW19 to SW18, SW20 to SW19, SW3 to SW2, SW21 to SW20, SW22 to SW21, SW23 to SW22, SW24 to SW23, SW25 to SW24, SW26 to SW25, SW27 to SW26, SW28 to SW27, SW29 to SW28, SW30 to SW29, SW4 to SW3, SW31 to SW30, SW32 to SW31, SW33 to SW32, SW34 to SW33, SW35 to SW34, SW36 to SW35, SW37 to SW36, SW38 to SW37, SW39 to SW38, SW40 to SW39, SW5 to SW4, SW41 to SW40, SW42 to SW41, SW43 to SW42, SW44 to SW43, SW45 to SW44, SW46 to SW45, SW47 to SW46, SW48 to SW47, SW49 to SW48, SW50 to SW49, SW6 to SW5, SW51 to SW50, SW52 to SW51, SW53 to SW52, SW54 to SW53, SW55 to SW54, SW56 to SW55, SW57 to SW56, SW58 to SW57, SW59 to SW58, SW60 to SW59, SW7 to SW6, SW61 to SW60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
Connections:
- net +3V3: now also C116.2, J2.5 (Pin_5)
- net GND: now also C100.1, C101.1, C116.1, C92.1, C93.1, C94.1, C95.1, C96.1, C97.1, C98.1, C99.1, J2.1 (Pin_1)
- net PREVGH: now also C98.2
- net PREVGL: now also C100.2
- net RST: now also J2.4 (Pin_4)
- net SWDCLK: now also J2.3 (Pin_3)
- net SWDIO: now also J2.2 (Pin_2)
- net at J4.5 (Pin_5): now also C93.2
- net at D204.1 (K), D205.2 (A): now also C121.1
- net at J4.4 (Pin_4): now also C92.2
- net at J4.20 (Pin_20): now also C97.2
- net at D203.2 (A), L2.2, Q4.3 (D): now also C121.2
- net at J4.19 (Pin_19): now also C96.2
- net at J4.15 (Pin_15): now also C94.2
- net at J4.22 (Pin_22): now also C99.2
- net at J4.18 (Pin_18): now also C95.2
- net at J4.24 (Pin_24): now also C101.2

Commit message: updated leds in schematics
Parts:
- removed D10, D100, D11, D113, D114, D115, D116, D117, D12, D13, D135, D136, D137, D138, D139, D14, D143, D144, D145, D146, D147, D148, D149, D15, D150, D151, D152, D158, D159, D16, D160, D161, D162, D17, D172, D173, D174, D175, D176, D18, D180, D181, D182, D183, D184, D185, D186, D187, D188, D189, D19, D190, D191, D192, D193, D194, D195, D196, D197, D198, D199, D2, D20, D200, D201, D202, D206, D207, D208, D209, D21, D22, D23, D24, D25, D26, D3, D39, D4, D40, D41, D42, D43, D5, D56, D57, D58, D59, D6, D60, D7, D73, D74, D75, D76, D77, D8, D9, D96, D97, D98, D99: SK6812MINI, LED_SMD:LED_WS2812B-MINI_PLCC4_3.5x3.5mm_P1.75mm, symbol marbastlib-various:WS2812B-MINI
- removed Q2: AO3400A, Package_TO_SOT_SMD:SOT-23, symbol Transistor_FET:AO3400A
- added LED1, LED10, LED100, LED101, LED102, LED103, LED11, LED12, LED13, LED14, LED15, LED16, LED17, LED18, LED19, LED2, LED20, LED21, LED22, LED23, LED24, LED25, LED26, LED27, LED28, LED29, LED3, LED30, LED31, LED32, LED33, LED34, LED35, LED36, LED37, LED38, LED39, LED4, LED40, LED41, LED42, LED43, LED44, LED45, LED46, LED47, LED48, LED49, LED5, LED50, LED51, LED52, LED53, LED54, LED55, LED56, LED57, LED58, LED59, LED6, LED60, LED61, LED62, LED63, LED64, LED65, LED66, LED67, LED68, LED69, LED7, LED70, LED71, LED72, LED73, LED74, LED75, LED77, LED78, LED79, LED8, LED80, LED81, LED82, LED83, LED84, LED85, LED86, LED87, LED88, LED89, LED9, LED90, LED91, LED92, LED93, LED94, LED95, LED96, LED97, LED98, LED99: MX_SK6812MINI-E, marbastlib-various:LED_6028R, symbol marbastlib-various:SK6812MINI-E
- added Q2: AO3401A, Package_TO_SOT_SMD:SOT-23, symbol Transistor_FET:AO3401A
- renumbered D35 to D10, D170 to D100, D171 to D101, D177 to D102, D178 to D103, D179 to D104, D203 to D105, D204 to D106, D205 to D107, D36 to D11, D37 to D12, D38 to D13, D44 to D14, D45 to D15, D46 to D16, D47 to D17, D48 to D18, D49 to D19, D27 to D2, D50 to D20, D51 to D21, D52 to D22, D53 to D23, D54 to D24, D55 to D25, D61 to D26, D62 to D27, D63 to D28, D64 to D29, D28 to D3, D65 to D30, D66 to D31, D67 to D32, D68 to D33, D69 to D34, D70 to D35, D71 to D36, D72 to D37, D78 to D38, D79 to D39, D29 to D4, D80 to D40, D81 to D41, D82 to D42, D83 to D43, D84 to D44, D85 to D45, D86 to D46, D87 to D47, D88 to D48, D89 to D49, D30 to D5, D90 to D50, D91 to D51, D92 to D52, D93 to D53, D94 to D54, D95 to D55, D101 to D56, D102 to D57, D103 to D58, D104 to D59, D31 to D6, D105 to D60, D106 to D61, D107 to D62, D108 to D63, D109 to D64, D110 to D65, D111 to D66, D112 to D67, D118 to D68, D119 to D69, D32 to D7, D120 to D70, D121 to D71, D122 to D72, D123 to D73, D124 to D74, D125 to D75, D126 to D76, D127 to D77, D128 to D78, D129 to D79, D33 to D8, D130 to D80, D131 to D81, D132 to D82, D133 to D83, D134 to D84, D140 to D85, D141 to D86, D142 to D87, D153 to D88, D154 to D89, D34 to D9, D155 to D90, D156 to D91, D157 to D92, D163 to D93, D164 to D94, D165 to D95, D166 to D96, D167 to D97, D168 to D98, D169 to D99, LED1 to LED76
Connections:
- net +VSW: now also Q2.2 (S)
- net GND: now also LED1.4 (VSS), LED10.4 (VSS), LED100.4 (VSS), LED101.4 (VSS), LED102.4 (VSS), LED103.4 (VSS), LED11.4 (VSS), LED12.4 (VSS), LED13.4 (VSS), LED14.4 (VSS), LED15.4 (VSS), LED16.4 (VSS), LED17.4 (VSS), LED18.4 (VSS), LED19.4 (VSS), LED2.4 (VSS), LED20.4 (VSS), LED21.4 (VSS), LED22.4 (VSS), LED23.4 (VSS), LED24.4 (VSS), LED25.4 (VSS), LED26.4 (VSS), LED27.4 (VSS), LED28.4 (VSS), LED29.4 (VSS), LED3.4 (VSS), LED30.4 (VSS), LED31.4 (VSS), LED32.4 (VSS), LED33.4 (VSS), LED34.4 (VSS), LED35.4 (VSS), LED36.4 (VSS), LED37.4 (VSS), LED38.4 (VSS), LED39.4 (VSS), LED4.4 (VSS), LED40.4 (VSS), LED41.4 (VSS), LED42.4 (VSS), LED43.4 (VSS), LED44.4 (VSS), LED45.4 (VSS), LED46.4 (VSS), LED47.4 (VSS), LED48.4 (VSS), LED49.4 (VSS), LED5.4 (VSS), LED50.4 (VSS), LED51.4 (VSS), LED52.4 (VSS), LED53.4 (VSS), LED54.4 (VSS), LED55.4 (VSS), LED56.4 (VSS), LED57.4 (VSS), LED58.4 (VSS), LED59.4 (VSS), LED6.4 (VSS), LED60.4 (VSS), LED61.4 (VSS), LED62.4 (VSS), LED63.4 (VSS), LED64.4 (VSS), LED65.4 (VSS), LED66.4 (VSS), LED67.4 (VSS), LED68.4 (VSS), LED69.4 (VSS), LED7.4 (VSS), LED70.4 (VSS), LED71.4 (VSS), LED72.4 (VSS), LED73.4 (VSS), LED74.4 (VSS), LED75.4 (VSS), LED77.4 (VSS), LED78.4 (VSS), LED79.4 (VSS), LED8.4 (VSS), LED80.4 (VSS), LED81.4 (VSS), LED82.4 (VSS), LED83.4 (VSS), LED84.4 (VSS), LED85.4 (VSS), LED86.4 (VSS), LED87.4 (VSS), LED88.4 (VSS), LED89.4 (VSS), LED9.4 (VSS), LED90.4 (VSS), LED91.4 (VSS), LED92.4 (VSS), LED93.4 (VSS), LED94.4 (VSS), LED95.4 (VSS), LED96.4 (VSS), LED97.4 (VSS), LED98.4 (VSS), LED99.4 (VSS)
- net UG_HL: now also LED1.3 (DIN)
- net UG_PWR: now also LED1.1 (VDD), LED10.1 (VDD), LED100.1 (VDD), LED101.1 (VDD), LED102.1 (VDD), LED103.1 (VDD), LED11.1 (VDD), LED12.1 (VDD), LED13.1 (VDD), LED14.1 (VDD), LED15.1 (VDD), LED16.1 (VDD), LED17.1 (VDD), LED18.1 (VDD), LED19.1 (VDD), LED2.1 (VDD), LED20.1 (VDD), LED21.1 (VDD), LED22.1 (VDD), LED23.1 (VDD), LED24.1 (VDD), LED25.1 (VDD), LED26.1 (VDD), LED27.1 (VDD), LED28.1 (VDD), LED29.1 (VDD), LED3.1 (VDD), LED30.1 (VDD), LED31.1 (VDD), LED32.1 (VDD), LED33.1 (VDD), LED34.1 (VDD), LED35.1 (VDD), LED36.1 (VDD), LED37.1 (VDD), LED38.1 (VDD), LED39.1 (VDD), LED4.1 (VDD), LED40.1 (VDD), LED41.1 (VDD), LED42.1 (VDD), LED43.1 (VDD), LED44.1 (VDD), LED45.1 (VDD), LED46.1 (VDD), LED47.1 (VDD), LED48.1 (VDD), LED49.1 (VDD), LED5.1 (VDD), LED50.1 (VDD), LED51.1 (VDD), LED52.1 (VDD), LED53.1 (VDD), LED54.1 (VDD), LED55.1 (VDD), LED56.1 (VDD), LED57.1 (VDD), LED58.1 (VDD), LED59.1 (VDD), LED6.1 (VDD), LED60.1 (VDD), LED61.1 (VDD), LED62.1 (VDD), LED63.1 (VDD), LED64.1 (VDD), LED65.1 (VDD), LED66.1 (VDD), LED67.1 (VDD), LED68.1 (VDD), LED69.1 (VDD), LED7.1 (VDD), LED70.1 (VDD), LED71.1 (VDD), LED72.1 (VDD), LED73.1 (VDD), LED74.1 (VDD), LED75.1 (VDD), LED77.1 (VDD), LED78.1 (VDD), LED79.1 (VDD), LED8.1 (VDD), LED80.1 (VDD), LED81.1 (VDD), LED82.1 (VDD), LED83.1 (VDD), LED84.1 (VDD), LED85.1 (VDD), LED86.1 (VDD), LED87.1 (VDD), LED88.1 (VDD), LED89.1 (VDD), LED9.1 (VDD), LED90.1 (VDD), LED91.1 (VDD), LED92.1 (VDD), LED93.1 (VDD), LED94.1 (VDD), LED95.1 (VDD), LED96.1 (VDD), LED97.1 (VDD), LED98.1 (VDD), LED99.1 (VDD), Q2.3 (D)
- net at Q1.3 (D), R9.2: now also Q2.1 (G)
- new net: LED38.2 (DOUT), LED43.3 (DIN)
- new net: LED33.2 (DOUT), LED38.3 (DIN)
- new net: LED10.2 (DOUT), LED15.3 (DIN)
- new net: LED10.3 (DIN), LED5.2 (DOUT)
- new net: LED58.2 (DOUT), LED63.3 (DIN)
- new net: LED53.2 (DOUT), LED58.3 (DIN)
- new net: LED23.2 (DOUT), LED28.3 (DIN)
- new net: LED18.2 (DOUT), LED23.3 (DIN)
- new net: LED30.2 (DOUT), LED35.3 (DIN)
- new net: LED25.2 (DOUT), LED30.3 (DIN)
- new net: LED94.2 (DOUT), LED98.3 (DIN)
- new net: LED89.2 (DOUT), LED94.3 (DIN)
- new net: LED59.2 (DOUT), LED64.3 (DIN)
- new net: LED54.2 (DOUT), LED59.3 (DIN)
- new net: LED39.2 (DOUT), LED44.3 (DIN)
- new net: LED34.2 (DOUT), LED39.3 (DIN)
- new net: LED101.2 (DOUT), LED3.3 (DIN)
- new net: LED101.3 (DIN), LED97.2 (DOUT)
- new net: LED80.2 (DOUT), LED85.3 (DIN)
- new net: LED74.2 (DOUT), LED80.3 (DIN)
- new net: LED71.2 (DOUT), LED77.3 (DIN)
- new net: LED66.2 (DOUT), LED71.3 (DIN)
- new net: LED84.2 (DOUT), LED89.3 (DIN)
- new net: LED79.2 (DOUT), LED84.3 (DIN)
- new net: LED50.2 (DOUT), LED55.3 (DIN)
- new net: LED45.2 (DOUT), LED50.3 (DIN)
- new net: LED70.2 (DOUT), LED75.3 (DIN)
- new net: LED65.2 (DOUT), LED70.3 (DIN)
- new net: LED86.2 (DOUT), LED91.3 (DIN)
- new net: LED43.2 (DOUT), LED48.3 (DIN)
- new net: LED28.2 (DOUT), LED33.3 (DIN)
- new net: LED37.2 (DOUT), LED42.3 (DIN)
- new net: LED32.2 (DOUT), LED37.3 (DIN)
- new net: LED14.3 (DIN), LED9.2 (DOUT)
- new net: LED4.2 (DOUT), LED9.3 (DIN)
- new net: LED95.2 (DOUT), LED99.3 (DIN)
- new net: LED90.2 (DOUT), LED95.3 (DIN)
- new net: LED103.2 (DOUT), LED5.3 (DIN)
- new net: LED21.2 (DOUT), LED26.3 (DIN)
- new net: LED16.2 (DOUT), LED21.3 (DIN)
- new net: LED67.2 (DOUT), LED72.3 (DIN)
- new net: LED62.2 (DOUT), LED67.3 (DIN)
- new net: LED13.2 (DOUT), LED18.3 (DIN)
- new net: LED13.3 (DIN), LED8.2 (DOUT)
- new net: LED60.2 (DOUT), LED65.3 (DIN)
- new net: LED85.2 (DOUT), LED90.3 (DIN)
- new net: LED82.2 (DOUT), LED87.3 (DIN)
- new net: LED77.2 (DOUT), LED82.3 (DIN)
- new net: LED103.3 (DIN), LED99.2 (DOUT)
- new net: LED57.2 (DOUT), LED62.3 (DIN)
- new net: LED61.2 (DOUT), LED66.3 (DIN)
- new net: LED56.2 (DOUT), LED61.3 (DIN)
- new net: LED48.2 (DOUT), LED53.3 (DIN)
- new net: LED83.2 (DOUT), LED88.3 (DIN)
- new net: LED78.2 (DOUT), LED83.3 (DIN)
- new net: LED40.2 (DOUT), LED45.3 (DIN)
- new net: LED35.2 (DOUT), LED40.3 (DIN)
- new net: LED102.2 (DOUT), LED4.3 (DIN)
- new net: LED102.3 (DIN), LED98.2 (DOUT)
- new net: LED51.2 (DOUT), LED56.3 (DIN)
- new net: LED46.2 (DOUT), LED51.3 (DIN)
- new net: LED81.2 (DOUT), LED86.3 (DIN)
- new net: LED100.3 (DIN), LED96.2 (DOUT)
- new net: LED92.2 (DOUT), LED96.3 (DIN)
- new net: LED72.2 (DOUT), LED78.3 (DIN)
- new net: LED87.2 (DOUT), LED92.3 (DIN)
- new net: LED2.2 (DOUT), LED7.3 (DIN)
- new net: LED100.2 (DOUT), LED2.3 (DIN)
- new net: LED64.2 (DOUT), LED69.3 (DIN)
- new net: LED24.2 (DOUT), LED29.3 (DIN)
- new net: LED19.2 (DOUT), LED24.3 (DIN)
- new net: LED49.2 (DOUT), LED54.3 (DIN)
- new net: LED44.2 (DOUT), LED49.3 (DIN)
- new net: LED73.2 (DOUT), LED79.3 (DIN)
- new net: LED68.2 (DOUT), LED73.3 (DIN)
- new net: LED3.2 (DOUT), LED8.3 (DIN)
- new net: LED17.2 (DOUT), LED22.3 (DIN)
- new net: LED12.2 (DOUT), LED17.3 (DIN)
- new net: LED1.2 (DOUT), LED6.3 (DIN)
- new net: LED26.2 (DOUT), LED31.3 (DIN)
- new net: LED93.2 (DOUT), LED97.3 (DIN)
- new net: LED42.2 (DOUT), LED47.3 (DIN)
- new net: LED14.2 (DOUT), LED19.3 (DIN)
- new net: LED11.2 (DOUT), LED16.3 (DIN)
- new net: LED11.3 (DIN), LED6.2 (DOUT)
- new net: LED27.2 (DOUT), LED32.3 (DIN)
- new net: LED22.2 (DOUT), LED27.3 (DIN)
- new net: LED69.2 (DOUT), LED74.3 (DIN)
- new net: LED12.3 (DIN), LED7.2 (DOUT)
- new net: LED41.2 (DOUT), LED46.3 (DIN)
- new net: LED36.2 (DOUT), LED41.3 (DIN)
- new net: LED47.2 (DOUT), LED52.3 (DIN)
- new net: LED52.2 (DOUT), LED57.3 (DIN)
- new net: LED75.2 (DOUT), LED81.3 (DIN)
- new net: LED88.2 (DOUT), LED93.3 (DIN)
- new net: LED20.2 (DOUT), LED25.3 (DIN)
- new net: LED15.2 (DOUT), LED20.3 (DIN)
- new net: LED29.2 (DOUT), LED34.3 (DIN)
- new net: LED55.2 (DOUT), LED60.3 (DIN)
- new net: LED63.2 (DOUT), LED68.3 (DIN)
- new net: LED31.2 (DOUT), LED36.3 (DIN)
